File: uBristleBot.brd (EAGLE design)
At the start: 25.4 x 25.4 mm, 41 parts, among them M1 MOTOR-304-103, M2 MOTOR-304-103, Q1 2N7002BKV, U2 MCP7383X.DFN, U3 LM3668, U4 TPS727XX.DSE

Commit message: Tweaked layout for GND plane
Routing:
- net N$8: track 23.9 -> 25.8 mm
- net GND: vias 28 -> 53
Changed lines of the file:
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@@
 <setting verticaltext="up"/>
 </settings>
-<grid distance="25" unitdist="mil" unit="mil" style="dots" multiple="2" display="yes" altdistance="5" altunitdist="mil" altunit="mil"/>
+<grid distance="25" unitdist="mil" unit="mil" style="dots" multiple="2" display="yes" altdistance="12.5" altunitdist="mil" altunit="mil"/>
 <layers>
 <layer number="1" name="Top" color="4" fill="1" visible="yes" active="yes"/>
@@
 <via x="17.4625" y="7.14375" extent="1-16" drill="0.3556"/>
 <via x="8.255" y="11.43" extent="1-16" drill="0.3556"/>
-<via x="10.795" y="11.43" extent="1-16" drill="0.3556"/>
 <via x="8.73125" y="7.14375" extent="1-16" drill="0.3556"/>
 <via x="7.77875" y="7.14375" extent="1-16" drill="0.3556"/>
@@
 <wire x1="16.0375" y1="8.1875" x2="17.2125" y2="8.1875" width="0.2032" layer="1"/>
 <wire x1="17.2125" y1="8.1875" x2="17.4625" y2="7.9375" width="0.2032" layer="1"/>
+<via x="8.763" y="16.129" extent="1-16" drill="0.3556"/>
+<via x="8.001" y="16.891" extent="1-16" drill="0.3556"/>
+<via x="6.985" y="13.335" extent="1-16" drill="0.3556"/>
+<via x="6.35" y="12.7" extent="1-16" drill="0.3556"/>
+<via x="5.715" y="12.065" extent="1-16" drill="0.3556"/>
+<via x="0.9525" y="14.9225" extent="1-16" drill="0.3556"/>
+<via x="0.9525" y="13.97" extent="1-16" drill="0.3556"/>
+<via x="0.9525" y="13.0175" extent="1-16" drill="0.3556"/>
+<via x="24.4475" y="14.9225" extent="1-16" drill="0.3556"/>
+<via x="24.4475" y="13.97" extent="1-16" drill="0.3556"/>
+<via x="24.4475" y="13.0175" extent="1-16" drill="0.3556"/>
+<via x="21.2725" y="14.9225" extent="1-16" drill="0.3556"/>
+<via x="21.2725" y="13.97" extent="1-16" drill="0.3556"/>
+<via x="21.2725" y="13.0175" extent="1-16" drill="0.3556"/>
+<via x="17.145" y="4.445" extent="1-16" drill="0.3556"/>
+<via x="18.415" y="0.9525" extent="1-16" drill="0.3556"/>
+<via x="18.415" y="1.905" extent="1-16" drill="0.3556"/>
+<via x="18.415" y="2.8575" extent="1-16" drill="0.3556"/>
+<via x="18.0975" y="4.445" extent="1-16" drill="0.3556"/>
+<via x="24.4475" y="6.985" extent="1-16" drill="0.3556"/>
+<via x="24.4475" y="5.715" extent="1-16" drill="0.3556"/>
+<via x="24.4475" y="4.445" extent="1-16" drill="0.3556"/>
+<via x="24.4475" y="8.255" extent="1-16" drill="0.3556"/>
+<via x="4.7625" y="7.3025" extent="1-16" drill="0.3556"/>
+<via x="3.81" y="7.3025" extent="1-16" drill="0.3556"/>
+<via x="2.8575" y="7.3025" extent="1-16" drill="0.3556"/>
 </signal>
 <signal name="5.0V">
@@
 <via x="7.77875" y="9.04875" extent="1-16" drill="0.3556"/>
 <wire x1="7.77875" y1="9.04875" x2="7.62" y2="9.2075" width="0.254" layer="16"/>
-<wire x1="7.62" y1="9.2075" x2="7.62" y2="16.51" width="0.254" layer="16"/>
+<wire x1="7.62" y1="9.2075" x2="7.62" y2="16.1925" width="0.254" layer="16"/>
 <wire x1="7.8525" y1="9.525" x2="7.77875" y2="9.45125" width="0.254" layer="1"/>
 <wire x1="7.77875" y1="9.45125" x2="7.77875" y2="9.04875" width="0.254" layer="1"/>
-<wire x1="7.62" y1="16.51" x2="5.08" y2="19.05" width="0.254" layer="16"/>
+<wire x1="7.62" y1="16.1925" x2="5.08" y2="18.7325" width="0.254" layer="16"/>
+<wire x1="5.08" y1="18.7325" x2="5.08" y2="19.05" width="0.254" layer="16"/>
 </signal>
 <signal name="BATT_DIV">
@@
 <wire x1="12.5175" y1="9.49" x2="12.25875" y2="9.49" width="0.254" layer="1"/>
 <wire x1="12.25875" y1="9.49" x2="12.065" y2="9.68375" width="0.254" layer="1"/>
-<wire x1="12.065" y1="9.68375" x2="11.7475" y2="10.00125" width="0.3048" layer="16"/>
-<wire x1="11.7475" y1="10.00125" x2="11.7475" y2="15.1765" width="0.3048" layer="16"/>
+<wire x1="12.065" y1="9.68375" x2="10.2235" y2="11.52525" width="0.3048" layer="16"/>
+<wire x1="10.2235" y1="11.52525" x2="10.2235" y2="16.7005" width="0.3048" layer="16"/>
 <contactref element="M1" pad="2"/>
 <wire x1="3.54" y1="23.1775" x2="4.14" y2="22.5775" width="0.4064" layer="1"/>
@@
 <wire x1="3.54" y1="23.1775" x2="3.09" y2="23.6275" width="0.4064" layer="1"/>
 <wire x1="3.09" y1="23.6275" x2="3.09" y2="24.4475" width="0.4064" layer="1"/>
-<wire x1="11.7475" y1="15.1765" x2="3.81" y2="23.114" width="0.3048" layer="16"/>
+<wire x1="10.2235" y1="16.7005" x2="3.81" y2="23.114" width="0.3048" layer="16"/>
 <wire x1="3.81" y1="23.114" x2="3.81" y2="24.13" width="0.3048" layer="16"/>
 <via x="3.81" y="24.13" extent="1-16" drill="0.3556"/>
@@
 <wire x1="14.2875" y1="8.73125" x2="14.2875" y2="9.525" width="0.254" layer="1"/>
 <wire x1="14.2875" y1="9.525" x2="14.44625" y2="9.68375" width="0.254" layer="1"/>
-<wire x1="14.44625" y1="9.68375" x2="13.81125" y2="10.31875" width="0.3048" layer="16"/>
-<wire x1="13.81125" y1="10.31875" x2="13.81125" y2="14.70025" width="0.3048" layer="16"/>
+<wire x1="16.637" y1="12.192" x2="14.478" y2="14.351" width="0.3048" layer="16"/>
 <contactref element="M2" pad="1"/>
 <wire x1="21.86" y1="23.1775" x2="21.26" y2="22.5775" width="0.4064" layer="1"/>
@@
 <wire x1="21.86" y1="23.1775" x2="22.31" y2="23.6275" width="0.4064" layer="1"/>
 <wire x1="22.31" y1="23.6275" x2="22.31" y2="24.4475" width="0.4064" layer="1"/>
-<wire x1="13.81125" y1="14.70025" x2="21.59" y2="22.479" width="0.3048" layer="16"/>
 <wire x1="21.59" y1="22.479" x2="21.59" y2="24.13" width="0.3048" layer="16"/>
 <via x="21.59" y="24.13" extent="1-16" drill="0.3556"/>
 <wire x1="21.59" y1="24.13" x2="21.9075" y2="24.4475" width="0.3048" layer="1"/>
 <wire x1="21.9075" y1="24.4475" x2="22.31" y2="24.4475" width="0.3048" layer="1"/>
+<wire x1="14.478" y1="14.351" x2="14.478" y2="15.367" width="0.3048" layer="16"/>
+<wire x1="14.478" y1="15.367" x2="21.59" y2="22.479" width="0.3048" layer="16"/>
+<wire x1="14.44625" y1="9.68375" x2="15.65275" y2="9.68375" width="0.3048" layer="16"/>
+<wire x1="15.65275" y1="9.68375" x2="16.637" y2="10.668" width="0.3048" layer="16"/>
+<wire x1="16.637" y1="10.668" x2="16.637" y2="12.192" width="0.3048" layer="16"/>
 </signal>
 <signal name="VBAT">
